File: pcb/blad.kicad_sch (KiCad schematic)
At the start: 91 parts, among them J1 Conn_01x04, J2 Conn_01x02_Pin, SW1 1U, SW10 1U, SW11 1U, SW12 1U, SW13 1.25U, SW14 1U, SW15 1U, SW16 1U, SW17 1U, SW18 1U, SW19 1U, SW2 1U, SW20 1U, SW21 1U, SW22 1U, SW23 1.75U, SW24 1U, SW25 1U, SW26 1U, SW27 1U, SW28 1U, SW29 1U, SW3 1U, SW30 1U, SW31 1U, SW32 1U, SW33 1.25U, SW34 1.25U, SW35 1U, SW36 1.25U, SW37 2.75U, SW38 1.25U, SW39 1U, SW4 1U, SW40 1.25U, SW41 1.75U, SW42 2.25U, SW5 1U, SW6 1U, SW7 1U, SW8 1U, SW9 1U, U1 HY0020

Commit message: Update PCB design for ANNA-B402
Parts:
- removed R1: 10k, Resistor_SMD:R_0402_1005Metric, symbol Device:R_Small
- removed TS1: RST, Button_Switch_SMD:SW_Push_SPST_NO_Alps_SKRK, symbol Switch:SW_SPST
- added J3: Conn_01x05, Connector_PinHeader_2.54mm:PinHeader_1x05_P2.54mm_Vertical, symbol Connector_Generic:Conn_01x05
- J1: value Conn_01x04 -> Conn_01x05
Connections:
- net +3V0: now also J3.2 (Pin_2)
- net GND: now also J3.1 (Pin_1)
- net SWDCLK: now also J3.4 (Pin_4)
- net SWDIO: now also J3.3 (Pin_3)
- net nRESET: now also J3.5 (Pin_5)
